File: Projects/01_Breadboard_Power_Supply/BreadBoardPowerSupply/BreadBoardPowerSupply.kicad_pcb (KiCad board)
At the start: 2 copper layers, 30.1 x 52.1 mm, 17 parts, among them J1 Barrel_Jack_Switch, J2 Conn_02x02_Odd_Even, J3 Conn_02x02_Odd_Even, SW1 SW_DPDT_x2, U1 LM7805_TO220

Commit message: Run DRC and fix errors - ignore courtyard errors for logos and graphics
Other:
- board text added: "470μF"
- board text added: "47μF"
- board text added: "560Ω"
- board text removed: "47 μF"
- board text removed: "470 μF"
- board text removed: "560 Ω"
