File: Projects/02_RPi_DHT_HAT/RaspberryPiHAT/RaspberryPiHAT.sch (KiCad schematic (older format))
At the start: 9 parts, among them J1 Raspberry_Pi_2_3, SW1 SW_DPST, U1 DHT22

Commit message: Project 2: Reroute nets and add copper fill for GND plane
Parts:
- R1, R2: value R -> 10 kΩ
- R3, R4: value R -> 330 Ω
Changed lines of the file:
@@
 P 6850 3600
 F 0 "R3" H 6920 3646 50  0000 L CNN
-F 1 "R" H 6920 3555 50  0000 L CNN
+F 1 "330 Ω" H 6920 3555 50  0000 L CNN
 F 2 "Resistor_SMD:R_0805_2012Metric" V 6780 3600 50  0001 C CNN
 F 3 "~" H 6850 3600 50  0001 C CNN
@@
 P 4100 3250
 F 0 "R2" V 3893 3250 50  0000 C CNN
-F 1 "R" V 3984 3250 50  0000 C CNN
+F 1 "10 kΩ" V 3984 3250 50  0000 C CNN
 F 2 "Resistor_SMD:R_0805_2012Metric" V 4030 3250 50  0001 C CNN
 F 3 "~" H 4100 3250 50  0001 C CNN
@@
 P 2600 3350
 F 0 "R1" H 2670 3396 50  0000 L CNN
-F 1 "R" H 2670 3305 50  0000 L CNN
+F 1 "10 kΩ" H 2670 3305 50  0000 L CNN
 F 2 "Resistor_SMD:R_0805_2012Metric" V 2530 3350 50  0001 C CNN
 F 3 "~" H 2600 3350 50  0001 C CNN
@@
 P 7850 3600
 F 0 "R4" H 7920 3646 50  0000 L CNN
-F 1 "R" H 7920 3555 50  0000 L CNN
+F 1 "330 Ω" H 7920 3555 50  0000 L CNN
 F 2 "Resistor_SMD:R_0805_2012Metric" V 7780 3600 50  0001 C CNN
 F 3 "~" H 7850 3600 50  0001 C CNN
