File: Projects/03_BACEE/BACEE/BACEE_4_Layer.kicad_pcb (KiCad board)
At the start: 4 copper layers, 44.7 x 28.4 mm, 17 parts, among them J1 Digital Pins, J2 Serial, J3 ICSP, J4 I2C, U1 DS1337_MLv1, U2 24LC1025, U3 24LC1025, U4 ATmega328P-AU, Y1 Crystal 32MHz, Y2 Crystal 16MHz

Commit message: Project 3: Route 4-layer board again
Parts:
- moved J4 2.03 mm to (229.4, 103.8)
- moved J1 1.97 mm to (216.4, 126.2)
- moved R2 1.51 mm to (211.3, 106.2)
- moved J2 1.08 mm to (216.4, 103.8)
- moved Y2 0.07 mm to (214.1, 109.7)
Routing:
- net GNDPWR: track 142.4 -> 176.5 mm
- net /Vcc: track 160.3 -> 133.3 mm, vias 0 -> 2
- net /RESET: track 44.6 -> 26.5 mm, vias 1 -> 2
- net /SCK: track 66.7 -> 81.0 mm
- net /ADDR2: track 27.4 -> 16.2 mm
- net Net-(U1-Pad2): track 7.36 -> 12.3 mm
- net /D8: track 19.7 -> 17.7 mm
- net /D5: track 14.5 -> 12.5 mm
- net /D7: track 17.9 -> 16.0 mm
- net /D6: track 16.2 -> 14.2 mm
- net /ADDR1: track 14.5 -> 16.1 mm, vias 0 -> 2
- net /D3: track 16.9 -> 18.6 mm
- net /SDA: track 44.9 -> 46.5 mm
- net /D4: track 18.6 -> 17.3 mm
- net Net-(C1-Pad1): track 36.9 -> 38.0 mm
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Other:
- board size 44.7 x 28.4 mm -> 42.4 x 26.4 mm

Commit message: Project 3: Add 4-layer board PCB as separate file and add copper fill for In2.Cu
Routing:
- added copper zone on In2.Cu, net GNDPWR
