File: Projects/03_BACEE/BACEE/BACEE_2_Layer.kicad_pcb (KiCad board)
At the start: 2 copper layers, 42.4 x 26.4 mm, 17 parts, among them J1 Digital Pins, J2 Serial, J3 ICSP, J4 I2C, U1 DS1337_MLv1, U2 24LC1025, U3 24LC1025, U4 ATmega328P-AU, Y1 Crystal 32MHz, Y2 Crystal 16MHz

Commit message: Project 3: Create copper fille for 2-layer board
Routing:
- removed copper zone on B.Cu, net GNDPWR
