File: Projects/03_BACEE/BACEE/BACEE.kicad_pcb (KiCad board)
At the start: 2 copper layers, 42.4 x 26.4 mm, 19 parts, among them J1 Digital Pins, J2 Serial, J3 ICSP, J4 I2C, U1 DS1337_MLv1, U2 24LC1025, U3 24LC1025, U4 ATmega328P-AU, Y1 XTL 32MHz, Y2 XTL 16MHz

Commit message: Project 3: Add new Ducky_Logo graphic footprint on B.SilkS
Parts:
- added G***: LOGO, Libraries:Ducky_Logo_1.8x1.8mm, B.Cu at (222.5, 114.6)
